Commit message: urdf modified

File: src/my_bot/description/imu.xacro (robot description, xacro)
@@ -4,5 +4,5 @@
         <parent link="chassis"/>
         <child link="imu_frame"/>
-        <origin xyz="0.3 0 0.03" rpy="0 0 0"/>
+        <origin xyz="0.52 0 0.22" rpy="0 0 0"/>
     </joint>
     <link name="imu_frame">

File: src/my_bot/description/lidar.xacro (robot description, xacro)
@@ -4,5 +4,5 @@
         <parent link="chassis"/>
         <child link="laser_frame"/>
-        <origin xyz="0.57 0 0.18" rpy="0 0 0"/>
+        <origin xyz="0.52 0 0.22" rpy="0 0 0"/>
     </joint>
     <link name="laser_frame">

File: src/my_bot/description/robot.urdf.xacro (robot description, xacro)
@@ -2,5 +2,5 @@
 <robot xmlns:xacro="http://www.ros.org/wiki/xacro"  name="robot">
     <xacro:arg name="use_ros2_control" default="true"/>
-    <xacro:arg name="sim_mode" default="true"/>
+    <xacro:arg name="sim_mode" default="false"/>
     <xacro:include filename="robot_core.xacro"/>
     <xacro:if value="$(arg use_ros2_control)">

File: src/my_bot/description/robot_core.xacro (robot description, xacro)
@@ -2,14 +2,14 @@
 <robot xmlns:xacro="http://www.ros.org/wiki/xacro" >
     <xacro:include filename="inertial_macros.xacro"/>
-    <xacro:property name="chassis_length" value="0.6"/>
-    <xacro:property name="chassis_width" value="0.6"/>
-    <xacro:property name="chassis_height" value="0.15"/>
+    <xacro:property name="chassis_length" value="0.63"/>
+    <xacro:property name="chassis_width" value="0.64"/>
+    <xacro:property name="chassis_height" value="0.20"/>
     <xacro:property name="chassis_mass" value="0.5"/>
     <xacro:property name="wheel_radius" value="0.0625"/>
     <xacro:property name="wheel_thickness" value="0.03"/>
     <xacro:property name="wheel_mass" value="1.0"/>
-    <xacro:property name="wheel_offset_x" value="0.3"/>
-    <xacro:property name="wheel_offset_y" value="0.326"/>
-    <xacro:property name="wheel_offset_z" value="-0.0625"/>
+    <xacro:property name="wheel_offset_x" value="0.315"/>
+    <xacro:property name="wheel_offset_y" value="0.34"/>
+    <xacro:property name="wheel_offset_z" value="0.0"/>
     <xacro:property name="caster_wheel_radius" value="0.05"/>
     <xacro:property name="caster_wheel_mass" value="0.5"/>
@@ -79,5 +79,5 @@
                 <box size="${chassis_length} ${chassis_width} ${chassis_height}"/>
             </geometry>
-            <material name="orange"/>
+            <material name="white"/>
         </visual>
         <collision>
@@ -92,5 +92,5 @@
     </link>
     <gazebo reference ="chassis">
-        <material>Gazebo/OrangeTransparent</material>
+        <material>Gazebo/WhiteTransparent</material>
     </gazebo>
     <!-- LEFT WHEEL LINK-->
@@ -106,5 +106,5 @@
                 <cylinder radius="${wheel_radius}" length="${wheel_thickness}"/>
             </geometry>
-            <material name="blue"/>
+            <material name="orange"/>
         </visual>
         <collision>
@@ -132,5 +132,5 @@
                 <cylinder radius="${wheel_radius}" length="${wheel_thickness}"/>
             </geometry>
-            <material name="blue"/>
+            <material name="orange"/>
         </visual>
         <collision>
@@ -157,5 +157,5 @@
                <sphere radius="${caster_wheel_radius}"/>
             </geometry>
-            <material name="white"/>
+            <material name="orange"/>
         </visual>
         <collision>

File: src/my_bot/description/ros2_control.xacro (robot description, xacro)
@@ -11,5 +11,5 @@
                 <param name="baud_rate">57600</param>
                 <param name="timeout">1000</param>
-                <param name="enc_counts_per_rev">3436</param>
+                <param name="enc_counts_per_rev">5035</param>
             </hardware>
             <joint name="left_wheel_joint">

Commit message: on dev_window

File: src/my_bot/description/imu.xacro (robot description, xacro)
@@ -4,5 +4,5 @@
         <parent link="chassis"/>
         <child link="imu_frame"/>
-        <origin xyz="0.52 0 0.22" rpy="0 0 0"/>
+        <origin xyz="0.52 0 0.20" rpy="0 0 0"/>
     </joint>
     <link name="imu_frame">

Commit message: localiztion test

File: src/my_bot/description/imu.xacro (robot description, xacro)
@@ -4,5 +4,5 @@
         <parent link="chassis"/>
         <child link="imu_frame"/>
-        <origin xyz="0.52 0 0.20" rpy="0 0 0"/>
+        <origin xyz="0.52 0 0.03" rpy="0 0 0"/>
     </joint>
     <link name="imu_frame">

File: src/my_bot/description/lidar.xacro (robot description, xacro)
@@ -4,5 +4,5 @@
         <parent link="chassis"/>
         <child link="laser_frame"/>
-        <origin xyz="0.52 0 0.22" rpy="0 0 0"/>
+        <origin xyz="0.52 0 0.30" rpy="0 0 0"/>
     </joint>
     <link name="laser_frame">

File: src/my_bot/description/ros2_control.xacro (robot description, xacro)
@@ -11,5 +11,6 @@
                 <param name="baud_rate">57600</param>
                 <param name="timeout">1000</param>
-                <param name="enc_counts_per_rev">5035</param>
+                <param name="enc_counts_per_rev">4805</param>
+                <!-- <param name="enc_counts_per_rev">5035</param> 5035 -->
             </hardware>
             <joint name="left_wheel_joint">
