Commit message: change

File: src/my_bot/description/lidar.xacro (robot description, xacro)
@@ -4,7 +4,35 @@
         <parent link="chassis"/>
         <child link="laser_frame"/>
-        <origin xyz="0.52 0 0.30" rpy="0 0 0"/>
+        <origin xyz="0.52 0 0.20" rpy="0 0 0"/>
     </joint>
     <link name="laser_frame">
+        <visual>
+            <geometry>
+                <cylinder radius="0.05" length="0.04"/>
+            </geometry>
+            <material name="black"/>
+        </visual>
+        <visual>
+            <origin xyz="0 0 -0.05"/>
+            <geometry>
+                <cylinder radius="0.01" length="0.1"/>
+            </geometry>
+            <material name="black"/>
+        </visual>
+        <collision>
+            <geometry>
+                <cylinder radius="0.05" length="0.04"/>
+            </geometry>
+        </collision>
+        <xacro:inertial_cylinder mass="0.1" length="0.04" radius="0.05">
+            <origin xyz="0 0 0" rpy="0 0 0"/>
+        </xacro:inertial_cylinder>
+    </link>
+     <joint name="laser_joint_filter" type="fixed">
+        <parent link="chassis"/>
+        <child link="laser_frame_filter"/>
+        <origin xyz="0.52 0 0.20" rpy="0 0 0"/>
+    </joint>
+    <link name="laser_frame_filter">
         <visual>
             <geometry>

File: src/my_bot/description/robot.urdf.xacro (robot description, xacro)
@@ -11,4 +11,4 @@
     </xacro:unless>
     <xacro:include filename="lidar.xacro" />
-    <xacro:include filename="imu.xacro" />
+    <!-- <xacro:include filename="imu.xacro" /> -->
 </robot>

File: src/my_bot/description/ros2_control.xacro (robot description, xacro)
@@ -7,10 +7,9 @@
                 <param name="left_wheel_name">left_wheel_joint</param>
                 <param name="right_wheel_name">right_wheel_joint</param>
-                <param name="loop_rate">30</param>
+                <param name="loop_rate">50</param>
                 <param name="device">/dev/ttyACM0</param>
                 <param name="baud_rate">57600</param>
                 <param name="timeout">1000</param>
                 <param name="enc_counts_per_rev">4805</param>
-                <!-- <param name="enc_counts_per_rev">5035</param> 5035 -->
             </hardware>
             <joint name="left_wheel_joint">
@@ -58,5 +57,5 @@
         <plugin name="gazebo_ros2_control" filename="libgazebo_ros2_control.so">
             <parameters>$(find my_bot)/config/my_controllers.yaml</parameters>
-            <!-- <parameters>$(find my_bot)/config/gaz_ros2_ctl_use_sim.yaml</parameters> -->
+            <parameters>$(find my_bot)/config/gaz_ros2_ctl_use_sim.yaml</parameters>
         </plugin>
     </gazebo>
